File: pcbs/MinimalSAMD21/MinimalSAMD21.kicad_pcb (KiCad board)
At the start: 2 copper layers, 55 x 35 mm, 15 parts, among them J2 Conn_01x14_Female, J3 Conn_01x14_Female, U1 AP2112K-3.3, U2 TQFP32_MC_MCH

Commit message: new design for minimal SAMD21 board
Parts:
- removed ? (x2): , 
- removed C4 1uF: 1uF, Capacitor_SMD:C_0805_2012Metric_Pad1.15x1.40mm_HandSolder
- removed C5 100nF: 100nF, Capacitor_SMD:C_0805_2012Metric_Pad1.15x1.40mm_HandSolder
- removed DEBUG: DEBUG, Connector_PinSocket_2.54mm:PinSocket_1x05_P2.54mm_Vertical
- removed R2: 330Ω, Resistor_SMD:R_0805_2012Metric_Pad1.15x1.40mm_HandSolder
- removed RESET: SW_Push, Joels KiCad Footprint Library:PTS526_SK15_SMTR2_LFS
- added C4: 1uF, Capacitor_SMD:C_0805_2012Metric_Pad1.18x1.45mm_HandSolder, F.Cu at (42.0, 81.3)
- added C5: 1uF, Capacitor_SMD:C_0805_2012Metric_Pad1.18x1.45mm_HandSolder, F.Cu at (36.9, 80.0)
- added C6: 2.2uF, Capacitor_SMD:C_0805_2012Metric_Pad1.18x1.45mm_HandSolder, F.Cu at (34.9, 76.0)
- added D1: NeoPixel_THT, Joels KiCad Footprint Library:LED_WS2812-2020, F.Cu at (43.7, 96.2)
- added D2: SD1206S020S1R0‎, Diode_SMD:D_1206_3216Metric, F.Cu at (39.3, 63.2)
- added DBG: DEBUG, Joels KiCad Footprint Library:CNC_3220-10-0300-00_SWD_Receptacle, F.Cu at (29.0, 60.5)
- added J4: Conn_01x07_Female, Connector_PinSocket_2.54mm:PinSocket_1x07_P2.54mm_Vertical, F.Cu at (48.3, 80.5)
- added RESET1: SW_Push, Joels KiCad Footprint Library:PTS526_SK15_SMTR2_LFS_Tactile_SW_5.2x5.2, F.Cu at (29.0, 72.5)
- added U3: MIC5225-3.3YM5, Joels KiCad Footprint Library:MIC5225-SOT23-5LD, F.Cu at (35.1, 69.9)
- C1, C2: footprint Capacitor_SMD:C_0805_2012Metric_Pad1.15x1.40mm_HandSolder -> Capacitor_SMD:C_0805_2012Metric_Pad1.18x1.45mm_HandSolder
- C3: value 100nF -> 1uF; footprint Capacitor_SMD:C_0805_2012Metric_Pad1.15x1.40mm_HandSolder -> Capacitor_SMD:C_0805_2012Metric_Pad1.18x1.45mm_HandSolder
- J2: value Conn_01x14_Female -> Conn_01x07_Female; footprint Connector_PinSocket_2.54mm:PinSocket_1x14_P2.54mm_Vertical -> Connector_PinSocket_2.54mm:PinSocket_1x07_P2.54mm_Vertical
- J3: value Conn_01x14_Female -> USB_B_Micro; footprint Connector_PinSocket_2.54mm:PinSocket_1x14_P2.54mm_Vertical -> Connector_USB:USB_Micro-B_Amphenol_10118194_Horizontal
- R1: footprint Resistor_SMD:R_0805_2012Metric_Pad1.15x1.40mm_HandSolder -> Resistor_SMD:R_0805_2012Metric_Pad1.20x1.40mm_HandSolder
- U1: value AP2112K-3.3 -> AP2112M-3.3
- U2: value TQFP32_MC_MCH -> ATSAMD21E18A-AF
- moved J3 162.9 mm to (38.0, 56.4), turned to 180 degrees
- moved C2 155.9 mm to (45.2, 75.8), turned to 0 degrees
- moved C1 154.0 mm to (43.1, 63.5)
- moved U1 152.4 mm to (46.0, 69.9), turned to 270 degrees
- moved J2 141.0 mm to (28.0, 80.5), turned to 0 degrees
- moved U2 134.5 mm to (38.1, 88.9), turned to 0 degrees
- moved C3 127.2 mm to (34.9, 63.5), turned to 180 degrees
- moved R1 105.3 mm to (44.3, 83.7), turned to 180 degrees
Connections:
- C3 pad 1: /*RESET -> +5V
- J2 pad 1: +3V3 -> /A0
- J2 pad 2: /PA00 -> /A1
- J2 pad 3: /PA01 -> /A2
- J2 pad 4: /PA02 -> /A3
- J2 pad 5: /PA03 -> /SDA
- J2 pad 6: /PA04 -> /SCL
- J2 pad 7: /PA05 -> /TX_A6
- J3 pad 1: +5V -> Net-(D2-Pad2)
- J3 pad 2: /PA14 -> /D-
- J3 pad 3: /PA15 -> /D+
- J3 pad 4: /PA16 -> Net-(J3-Pad4)
- J3 pad 5: /PA17 -> GND
- J3 pad 6: /PA18 -> GND
- R1 pad 2: /*RESET -> /~RESET
- U2 pad 1: /PA00 -> Net-(U2-Pad1)
- U2 pad 11: /PA08 -> Net-(U2-Pad11)
- U2 pad 12: /PA09 -> /MISO
- U2 pad 13: /PA10 -> /MOSI
- U2 pad 14: /PA11 -> /SCK
- U2 pad 15: /PA14 -> Net-(U2-Pad15)
- U2 pad 16: /PA15 -> /NEO_PWR
- U2 pad 17: /PA16 -> /SDA
- U2 pad 18: /PA17 -> /SCL
- U2 pad 19: /PA18 -> /NEOPIX
- U2 pad 2: /PA01 -> Net-(U2-Pad2)
- U2 pad 20: /PA19 -> Net-(U2-Pad20)
- U2 pad 21: /PA22 -> Net-(U2-Pad21)
- U2 pad 22: /PA23 -> Net-(U2-Pad22)
- U2 pad 23: /PA24 -> /D-
- U2 pad 24: /PA25 -> /D+
- U2 pad 25: /PA27 -> Net-(U2-Pad25)
- U2 pad 26: /*RESET -> /~RESET
- U2 pad 27: /PA28 -> Net-(U2-Pad27)
- U2 pad 3: /PA02 -> /A0
- U2 pad 4: /PA03 -> /A1
- U2 pad 5: /PA04 -> /A2
- U2 pad 6: /PA05 -> /A3
- U2 pad 7: /PA06 -> /TX_A6
- U2 pad 8: /PA07 -> /RX_A7
Routing:
- net GND: track 17.6 -> 89.0 mm, vias 14 -> 4
- net /*RESET: track 53.5 -> 0.00 mm, vias 4 -> 0
- net +3V3: track 112.7 -> 71.5 mm, vias 2 -> 0
- net /~RESET: track 0.00 -> 40.1 mm, vias 0 -> 2
- net /D+: track 0.00 -> 35.8 mm, vias 0 -> 2
- net /D-: track 0.00 -> 35.8 mm, vias 0 -> 2
- net /PA14: track 25.9 -> 0.00 mm
- net /PA11: track 25.7 -> 0.00 mm
- net /PA10: track 23.4 -> 0.00 mm
- net +5V: track 18.2 -> 41.0 mm
- net /PA15: track 22.1 -> 0.00 mm
- net /PA07: track 21.7 -> 0.00 mm
- net /PA09: track 21.2 -> 0.00 mm
- net /PA06: track 21.0 -> 0.00 mm
- net /RX_A7: track 0.00 -> 20.7 mm
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Other:
- board size 55 x 35 mm -> 24.5 x 46.5 mm
- rule pad_to_mask_clearance: 0.051 -> 0
- board text added: "ATSAMD21E DEV BOARD 2.0 JOEL SPOLSKY DEC 8, 2021 QtPy compatible? Thanks to Lady Ada"
- board text added: "RESET"
- board text removed: "+3V3 OUT"
- board text removed: "+5V IN"
- board text removed: "3V3"
- board text removed: "ATSAMD21E BREAKOUT WITH POWER AND RESET"
- board text removed: "BLINKY PROTO 0.1"
- board text removed: "GND"
- board text removed: "PA00"
- board text removed: "PA01"
- board text removed: "PA02"
- board text removed: "PA03"
- board text removed: "PA04"
- board text removed: "PA05"
- board text removed: "PA06"
- board text removed: "PA07"
- board text removed: "PA08"
- board text removed: "PA09"
- board text removed: "PA10"
- board text removed: "PA11"
- board text removed: "PA14"
- board text removed: "PA15"
- board text removed: "PA16"
- board text removed: "PA17"
- board text removed: "PA18"
- board text removed: "PA19"
- board text removed: "PA22"
- board text removed: "PA23"
- board text removed: "PA24"
- board text removed: "PA25"
- board text removed: "PA27"
- board text removed: "PA28"
- board text removed: "RESET*"
- board text removed: "SWCLK"
- board text removed: "SWDIO"
- board text removed: "●"
