File: pcbs/MinimalSAMD21/MinimalSAMD21.sch (KiCad schematic (older format))
At the start: 13 parts, among them J1 DEBUG, J2 Conn_01x14_Female, J3 Conn_01x14_Female, U1 AP2112K-3.3, U2 ATSAMD21E18A-AF

Commit message: new design for minimal SAMD21 board
Parts:
- removed J3: Conn_01x14_Female, Connector_PinSocket_2.54mm:PinSocket_1x14_P2.54mm_Vertical, symbol Connector:Conn_01x14_Female
- removed R2: 330Ω, Resistor_SMD:R_0805_2012Metric_Pad1.15x1.40mm_HandSolder, symbol Device:R
- added C6: 2.2uF, Capacitor_SMD:C_0805_2012Metric_Pad1.18x1.45mm_HandSolder, symbol Device:C
- added D1: NeoPixel_THT, Joels KiCad Footprint Library:LED_WS2812-2020, symbol LED:NeoPixel_THT
- added D2: SD1206S020S1R0‎, Diode_SMD:D_1206_3216Metric, symbol Device:D
- added J3: USB_B_Micro, Connector_USB:USB_Micro-B_Amphenol_10118194_Horizontal, symbol Connector:USB_B_Micro
- added J4: Conn_01x07_Female, Connector_PinSocket_2.54mm:PinSocket_1x07_P2.54mm_Vertical, symbol Connector:Conn_01x07_Female
- added U3: MIC5225-3.3YM5, Joels KiCad Footprint Library:MIC5225-SOT23-5LD, symbol Joels_KiCad_Symbol_Library:MIC5225-3.3YM5
- C1, C2, C4: footprint Capacitor_SMD:C_0805_2012Metric_Pad1.15x1.40mm_HandSolder -> Capacitor_SMD:C_0805_2012Metric_Pad1.18x1.45mm_HandSolder
- C3, C5: value 100nF -> 1uF; footprint Capacitor_SMD:C_0805_2012Metric_Pad1.15x1.40mm_HandSolder -> Capacitor_SMD:C_0805_2012Metric_Pad1.18x1.45mm_HandSolder
- J1: footprint Connector_PinSocket_2.54mm:PinSocket_1x05_P2.54mm_Vertical -> Joels KiCad Footprint Library:CNC_3220-10-0300-00_SWD_Receptacle; symbol Connector:Conn_01x05_Female -> Connector:Conn_01x10_Female
- J2: value Conn_01x14_Female -> Conn_01x07_Female; footprint Connector_PinSocket_2.54mm:PinSocket_1x14_P2.54mm_Vertical -> Connector_PinSocket_2.54mm:PinSocket_1x07_P2.54mm_Vertical; symbol Connector:Conn_01x14_Female -> Connector:Conn_01x07_Female
- R1: footprint Resistor_SMD:R_0805_2012Metric_Pad1.15x1.40mm_HandSolder -> Resistor_SMD:R_0805_2012Metric_Pad1.20x1.40mm_HandSolder
- RESET1: renamed from SWRESET; footprint Connector_PinSocket_2.54mm:PinSocket_1x02_P2.54mm_Vertical -> Joels KiCad Footprint Library:PTS526_SK15_SMTR2_LFS_Tactile_SW_5.2x5.2
- U1: value AP2112K-3.3 -> AP2112M-3.3
Connections:
- net +3V3: now also J1.1 (Pin_1), C6.1, J4.3 (Pin_3), U3.5 (OUT); no longer J1.2 (Pin_2), J2.1 (Pin_1)
- net +5V: now also C3.1, D2.1 (K), J4.1 (Pin_1), U3.1 (IN), U3.3 (EN)
- net GND: now also J1.2 (Pin_2), J1.5 (Pin_5), RESET1.4, C6.2, D1.2 (GND), J3.5 (GND), J3.6 (Shield), J4.2 (Pin_2), U3.2 (GND); no longer J2.14 (Pin_14)
- net SWCLK: now also J1.9 (Pin_9); no longer J1.5 (Pin_5)
- net SWDIO: now also J1.10 (Pin_10); no longer J1.4 (Pin_4)
- net ~RESET: now reaches RESET1.1
- net ~RESET: now also J1.6 (Pin_6), R1.2, RESET1.2, U2.26 (~RESET)
- removed net *RESET: C3.1, J1.1 (Pin_1), R1.2, U2.26 (~RESET)
- net PA00: no longer names the net of U2.1 (PA00)
- net PA00: no longer J2.2 (Pin_2)
- net PA01: no longer names the net of U2.2 (PA01)
- net PA01: no longer J2.3 (Pin_3)
- net PA02 renamed A0
- net A0: now also J2.1 (Pin_1); no longer J2.4 (Pin_4)
- net PA03 renamed A1
- net A1: now also J2.2 (Pin_2); no longer J2.5 (Pin_5)
- net PA04 renamed A2
- net A2: now also J2.3 (Pin_3); no longer J2.6 (Pin_6)
- net PA05 renamed A3
- net A3: now also J2.4 (Pin_4); no longer J2.7 (Pin_7)
- net PA06 renamed TX_A6
- net TX_A6: now also J2.7 (Pin_7); no longer J2.8 (Pin_8)
- net PA07 renamed RX_A7
- net RX_A7: now also J4.7 (Pin_7); no longer J2.9 (Pin_9)
- net PA08: no longer names the net of U2.11 (PA08)
- net PA08: no longer J2.10 (Pin_10)
- net PA09 renamed MISO
- net MISO: now also J4.5 (Pin_5); no longer J2.11 (Pin_11)
- net PA10 renamed MOSI
- net MOSI: now also J4.4 (Pin_4); no longer J2.12 (Pin_12)
- net PA11 renamed SCK
- net SCK: now also J4.6 (Pin_6); no longer J2.13 (Pin_13)
- net PA14: no longer names the net of U2.15 (PA14)
- net PA15 renamed NEO_PWR
- net NEO_PWR: now also D1.3 (VDD)
- net PA16 renamed SDA
- net SDA: now also J2.5 (Pin_5)
- net PA17 renamed SCL
- net SCL: now also J2.6 (Pin_6)
- net PA18 renamed NEOPIX
- net NEOPIX: now also D1.4 (DIN)
- net PA19: no longer names the net of U2.20 (PA19)
- net PA22: no longer names the net of U2.21 (PA22)
- net PA23: no longer names the net of U2.22 (PA23)
- net PA24 renamed D-
- net D-: now also J3.2 (D-)
- net PA25 renamed D+
- net D+: now also J3.3 (D+)
- net PA27: no longer names the net of U2.25 (PA27)
- net PA28: no longer names the net of U2.27 (PA28)
- new net: D2.2 (A), J3.1 (VBUS)
- no-connect marks 2 -> 15
