File: pcbs/ClonedESP32DevBoard/ClonedESP32DevBoard.sch (KiCad schematic (older format))
At the start: 30 parts, among them IC1 ESP32-C3-MINI-1-H4, J1 Adafruit_CP2104_Friend, J3 HDR1, J4 HDR2, Q1 KSC3265YMTF, Q2 KSC3265YMTF, SW1 BOOT, SW2 RST, SW3 JS202011JCQN, U1 AP2112M-3.3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

Commit message: why is kicad so annoying
Parts:
- IC1: symbol Joels_KiCad_Symbol_Library:ESP32-C3-MINI-1-H4 -> ClonedESP32DevBoard-rescue:ESP32-C3-MINI-1-H4-Joels_KiCad_Symbol_Library
- J1: symbol Joels_KiCad_Symbol_Library:Adafruit_CP2104_Friend -> ClonedESP32DevBoard-rescue:Adafruit_CP2104_Friend-Joels_KiCad_Symbol_Library
- U2: symbol Joels_KiCad_Symbol_Library:MIC5225-3.3YM5 -> ClonedESP32DevBoard-rescue:MIC5225-3.3YM5-Joels_KiCad_Symbol_Library
Other:
- note added: "warning\nincorrect\npinout"
Changed lines of the file:
@@
 $EndDescr
 $Comp
-L Joels_KiCad_Symbol_Library:Adafruit_CP2104_Friend J1
+L ClonedESP32DevBoard-rescue:Adafruit_CP2104_Friend-Joels_KiCad_Symbol_Library J1
 U 1 1 61BD45F6
 P 1850 1450
@@
 	1050 6750 1050 5100
 $Comp
-L Joels_KiCad_Symbol_Library:MIC5225-3.3YM5 U2
+L ClonedESP32DevBoard-rescue:MIC5225-3.3YM5-Joels_KiCad_Symbol_Library U2
 U 1 1 61C1FF3E
 P 6750 5550
@@
 	8100 3750 7850 3750
 $Comp
-L Joels_KiCad_Symbol_Library:ESP32-C3-MINI-1-H4 IC1
+L ClonedESP32DevBoard-rescue:ESP32-C3-MINI-1-H4-Joels_KiCad_Symbol_Library IC1
 U 1 1 61D1A13C
 P 11400 1650
@@
 Wire Wire Line
 	9250 6750 9250 6850
+Text Notes 1050 4450 0    276  ~ 0
+warning\nincorrect\npinout
 $EndSCHEMATC
