File: pcbs/ledtrix/ledtrix for blinky.sch (KiCad schematic (older format))
At the start: 178 parts, among them IC1 TSOP36438TT, J1 JACK IN, J3 CA1-9, J4 CB1-9, Q1 PMBT2222A,215, SW1 TACTILE, U1 ATSAMD21E17, U2 MIC5225-3.3YM5, U4 IS31FL3731-SALS2

Commit message: routing this board here
Parts:
- removed BT1, BT2: CR2032, Joels KiCad Footprint Library:BatteryHolder_Keystone_3034_Minimum_Pad, symbol Device:Battery_Cell
- removed C1: 100uF 6.3V, Capacitor_SMD:C_1206_3216Metric, symbol Device:C
- removed C10, C11: 10uF, Capacitor_SMD:C_0603_1608Metric, symbol Device:C_Small
- removed C2, C7: 1uF, Capacitor_SMD:C_0603_1608Metric, symbol Device:C
- removed C3, C4, C8: 0.1uF, Capacitor_SMD:C_0603_1608Metric, symbol Device:C
- removed C5: 1.0uF, Capacitor_SMD:C_0603_1608Metric, symbol Device:C
- removed C6: 2.2uF, Capacitor_SMD:C_0603_1608Metric, symbol Device:C
- removed C9: 0.1uF, Capacitor_SMD:C_0603_1608Metric, symbol Device:C_Small
- removed D145: IR LED, LED_SMD:LED_0805_2012Metric, symbol Device:LED
- removed IC1: TSOP36438TT, Joels KiCad Footprint Library:TSOP36438TT, symbol Joels_KiCad_Symbol_Library:TSOP36438TT
- removed J1: JACK IN, Joels KiCad Footprint Library:SOIC_clipProgSmall, symbol Connector_Generic:Conn_02x04_Counter_Clockwise
- removed J3: CA1-9, Connector_PinHeader_2.54mm:PinHeader_1x09_P2.54mm_Vertical, symbol Connector:Conn_01x09_Female
- removed J4: CB1-9, Connector_PinHeader_2.54mm:PinHeader_1x09_P2.54mm_Vertical, symbol Connector:Conn_01x09_Female
- removed Q1: PMBT2222A,215, Joels KiCad Footprint Library:NXP-TO-236AB-0-0-0, symbol Joels_KiCad_Symbol_Library:PMBT2222A,215
- removed R1: 10kΩ, Resistor_SMD:R_0603_1608Metric, symbol Device:R
- removed R10, R5, R6, R7, R8, R9: 20K, Resistor_SMD:R_0603_1608Metric, symbol Device:R
- removed R2: 330Ω, Resistor_SMD:R_0603_1608Metric, symbol Device:R
- removed R3: 47Ω, Resistor_SMD:R_0603_1608Metric, symbol Device:R
- removed R4: 470Ω, Resistor_SMD:R_0603_1608Metric, symbol Device:R
- removed S1: JS202011JCQN, Joels KiCad Footprint Library:CK-JS202011JCQN, symbol Joels_KiCad_Symbol_Library:JS202011JCQN
- removed SW1: TACTILE, Joels KiCad Footprint Library:TL9320AF400QG, symbol Switch:SW_SPST
- removed U1: ATSAMD21E17, Joels KiCad Footprint Library:ATSAMD21E17_32Pin_TQFP, symbol Joels_KiCad_Symbol_Library:ATSAMD21E18A-AF
- removed U2: MIC5225-3.3YM5, Joels KiCad Footprint Library:MIC5225-SOT23-5LD, symbol Joels_KiCad_Symbol_Library:MIC5225-3.3YM5
- removed U4: IS31FL3731-SALS2, Package_SO:SSOP-28_5.3x10.2mm_P0.65mm, symbol Driver_LED:IS31FL3731-SA
Connections:
- net labels removed: +3.3V, +5V, A0, A1, A2, A3, A6, A7, CFILT, GND, SCL, SDA, SWCLK, SWDIO, VBUS, ~RESET
- wire segments 766 -> 610
- no-connect marks 22 -> 0
Other:
- note removed: "BATTERY AND SWITCH"
- note removed: "CHARLIEPLEX MATRIX LED DRIVER"
- note removed: "CONTROL"
- note removed: "IR RECEIVER"
- note removed: "IR TRANSMITTER"
- note removed: "LED MATRIX"
- note removed: "LINEAR REGULATOR"
- note removed: "MCU - ATSAMD21E17"
- note removed: "POWER - ref datasheet 38.2"
- note removed: "RESET - ref datasheet 38.4"
- note removed: "SOIC-8 CLIP FLASH AND TEST"
