File: pcbs/blinky/blinky.kicad_pcb (KiCad board)
At the start: 4 copper layers, 135 x 97 mm, 178 parts, among them J1 JACK IN, J3 CA1-9, J4 CB1-9, Q1 PMBT2222A,215, SW1 TACTILE, SW2 JS202011JCQN, U1 ATSAMD21E17, U2 MIC5225-3.3YM5, U3 TSOP36438TT, U4 IS31FL3731-SALS2

Commit message: some 3d models
Parts:
- turned U3 to 90 degrees
Other:
- board text added: "OFF"
Changed lines of the file:
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@@
   (general
     (thickness 1.6)
-    (drawings 19)
+    (drawings 20)
     (tracks 946)
     (zones 0)
@@
       (rotate (xyz 0 0 0))
     )
+    (model "/Users/spolsky/Dropbox/src/KiCad Libraries/3d Models/SOT-23-5_M5_MCH.step"
+      (at (xyz 0 0 0))
+      (scale (xyz 1 1 1))
+      (rotate (xyz 0 0 0))
+    )
   )
   (module "Joels KiCad Footprint Library:ATSAMD21E17_32Pin_TQFP" (layer F.Cu)
@@
     (pad 2 smd rect (at 4.0513 0 90) (size 1.7018 2.6924) (layers F.Cu F.Paste F.Mask)
       (net 3 GND))
+    (model "/Users/spolsky/Dropbox/src/KiCad Libraries/3d Models/TL9320AF400QG.stp"
+      (at (xyz 0 0 0))
+      (scale (xyz 1 1 1))
+      (rotate (xyz 0 0 0))
+    )
   )
   (module "Joels KiCad Footprint Library:CK-JS202011JCQN" (layer F.Cu)
@@
     (pad 7 smd rect (at 1.2 2.5) (size 1.6 1) (layers F.Cu F.Paste F.Mask)
       (net 65 "Net-(SW2-Pad7)"))
+    (model "/Users/spolsky/Dropbox/src/KiCad Libraries/3d Models/JS202011JCQN.stp"
+      (at (xyz 0 0 0))
+      (scale (xyz 1 1 1))
+      (rotate (xyz 90 180 90))
+    )
   )
   (module Resistor_SMD:R_0603_1608Metric (layer F.Cu)
@@
       (rotate (xyz 0 0 0))
     )
+    (model "/Users/spolsky/Dropbox/src/KiCad Libraries/3d Models/SOT23_NEX.step"
+      (at (xyz 0 0 0))
+      (scale (xyz 1 1 1))
+      (rotate (xyz 0 0 0))
+    )
   )
   (module Connector_PinHeader_2.54mm:PinHeader_1x09_P2.54mm_Vertical (layer F.Cu)
@@
     (pad 1 thru_hole rect (at 0 0 270) (size 1.7 1.7) (drill 1) (layers *.Cu *.Mask)
       (net 31 /CB1))
-    (model ${KISYS3DMOD}/Connector_PinHeader_2.54mm.3dshapes/PinHeader_1x09_P2.54mm_Vertical.wrl
-      (at (xyz 0 0 0))
-      (scale (xyz 1 1 1))
-      (rotate (xyz 0 0 0))
-    )
   )
   (module Connector_PinHeader_2.54mm:PinHeader_1x09_P2.54mm_Vertical (layer F.Cu)
@@
     (pad 1 thru_hole rect (at 0 0 270) (size 1.7 1.7) (drill 1) (layers *.Cu *.Mask)
       (net 22 /CA1))
-    (model ${KISYS3DMOD}/Connector_PinHeader_2.54mm.3dshapes/PinHeader_1x09_P2.54mm_Vertical.wrl
-      (at (xyz 0 0 0))
-      (scale (xyz 1 1 1))
-      (rotate (xyz 0 0 0))
-    )
   )
   (module "Joels KiCad Footprint Library:SOIC_clipProgSmall" (layer F.Cu)
@@
   )
   (module "Joels KiCad Footprint Library:TSOP36438TT" (layer F.Cu)
-    (at 102.872 106.504)
+    (at 102.872 106.504 90)
     (descr TSOP36438TT-2)
     (tags "Integrated Circuit")
     (attr smd)
-    (fp_text reference U3 (at 0 -0.8) (layer F.SilkS)
+    (fp_text reference U3 (at 0 -0.8 90) (layer F.SilkS)
       (effects (font (size 1.27 1.27) (thickness 0.254)))
     )
-    (fp_text value TSOP36438TT (at 0 0.775) (layer F.SilkS) hide
+    (fp_text value TSOP36438TT (at 0 0.775 90) (layer F.SilkS) hide
       (effects (font (size 1.27 1.27) (thickness 0.254)))
     )
@@
     (fp_line (start 3.75 -2) (end 3.75 2) (layer F.Fab) (width 0.2))
     (fp_line (start -3.75 -2) (end 3.75 -2) (layer F.Fab) (width 0.2))
-    (fp_text user %R (at 0 0.775) (layer F.Fab)
+    (fp_text user %R (at 0 0.775 90) (layer F.Fab)
       (effects (font (size 1.27 1.27) (thickness 0.254)))
     )
@@
     (fp_arc (start -2.05 3.5) (end -2 3.5) (angle -180) (layer F.SilkS) (width 0.2))
     (fp_arc (start -2.05 3.5) (end -2.1 3.5) (angle -180) (layer F.SilkS) (width 0.2))
-    (pad 1 smd rect (at -1.905 1.3) (size 0.9 2.2) (layers F.Cu F.Paste F.Mask)
+    (pad 1 smd rect (at -1.905 1.3 90) (size 0.9 2.2) (layers F.Cu F.Paste F.Mask)
       (net 3 GND))
-    (pad 2 smd rect (at -0.635 1.3) (size 0.9 2.2) (layers F.Cu F.Paste F.Mask)
+    (pad 2 smd rect (at -0.635 1.3 90) (size 0.9 2.2) (layers F.Cu F.Paste F.Mask)
       (net 63 "Net-(U3-Pad2)"))
-    (pad 3 smd rect (at 0.635 1.3) (size 0.9 2.2) (layers F.Cu F.Paste F.Mask)
+    (pad 3 smd rect (at 0.635 1.3 90) (size 0.9 2.2) (layers F.Cu F.Paste F.Mask)
       (net 6 "Net-(C7-Pad1)"))
-    (pad 4 smd rect (at 1.905 1.3) (size 0.9 2.2) (layers F.Cu F.Paste F.Mask)
+    (pad 4 smd rect (at 1.905 1.3 90) (size 0.9 2.2) (layers F.Cu F.Paste F.Mask)
       (net 8 /A1))
-    (model TSOP36438TT.stp
+    (model "/Users/spolsky/Dropbox/src/KiCad Libraries/3d Models/82826SMD.STP"
       (at (xyz 0 0 0))
       (scale (xyz 1 1 1))
@@
     )
   )
+  (gr_text OFF (at 56.94 140.559) (layer F.SilkS)
+    (effects (font (size 1 1) (thickness 0.15)))
+  )
   (gr_text "CR2032 BATTERY\nFLAT SIDE UP" (at 72.8785 117.572 90) (layer B.SilkS)
     (effects (font (size 1.5 1.5) (thickness 0.2)) (justify mirror))
   )
-  (gr_text ON (at 80.8795 177.262 180) (layer F.SilkS)
+  (gr_text ON (at 56.813 135.479) (layer F.SilkS)
     (effects (font (size 1 1) (thickness 0.15)))
   )
