File: pcbs/blinky/blinky.sch (KiCad schematic (older format))
At the start: 39 parts, among them J1 Debug, Q1 PMBT2222A,215, SW1 TACTILE, SW2 POWER, U1 ATSAMD21E17, U2 MIC5225-3.3YM5, U3 TSOP75438WTT, U4 IS31FL3731-SALS2

Commit message: blinky version 1 PCB design is done!
Parts:
- added D1.1, D1.10, D1.11, D1.12, D1.13, D1.14, D1.15, D1.16, D1.2, D1.3, D1.4, D1.5, D1.6, D1.7, D1.8, D1.9, D2.1, D2.10, D2.11, D2.12, D2.13, D2.14, D2.15, D2.16, D2.2, D2.3, D2.4, D2.5, D2.6, D2.7, D2.8, D2.9, D3.1, D3.10, D3.11, D3.12, D3.13, D3.14, D3.15, D3.16, D3.2, D3.3, D3.4, D3.5, D3.6, D3.7, D3.8, D3.9, D4.1, D4.10, D4.11, D4.12, D4.13, D4.14, D4.15, D4.16, D4.2, D4.3, D4.4, D4.5, D4.6, D4.7, D4.8, D4.9, D5.1, D5.10, D5.11, D5.12, D5.13, D5.14, D5.15, D5.16, D5.2, D5.3, D5.4, D5.5, D5.6, D5.7, D5.8, D5.9, D6.1, D6.10, D6.11, D6.12, D6.13, D6.14, D6.15, D6.16, D6.2, D6.3, D6.4, D6.5, D6.6, D6.7, D6.8, D6.9, D7.1, D7.10, D7.11, D7.12, D7.13, D7.14, D7.15, D7.16, D7.2, D7.3, D7.4, D7.5, D7.6, D7.7, D7.8, D7.9, D8.1, D8.10, D8.11, D8.12, D8.13, D8.14, D8.15, D8.16, D8.2, D8.3, D8.4, D8.5, D8.6, D8.7, D8.8, D8.9, D9.1, D9.10, D9.11, D9.12, D9.13, D9.14, D9.15, D9.16, D9.2, D9.3, D9.4, D9.5, D9.6, D9.7, D9.8, D9.9: LED, Joels KiCad Footprint Library:LED_0603_For_Blinky, symbol Device:LED
- added J2: NEOPIXEL, Joels KiCad Footprint Library:Debug_Pad_01x03, symbol Connector_Generic:Conn_01x03
- BT1, BT2: footprint Battery:BatteryHolder_Keystone_3034_1x20mm -> Joels KiCad Footprint Library:BatteryHolder_Keystone_3034_Minimum_Pad
- J1: value Debug -> JACK IN
Connections:
- net labels added: NEOPIX, NEOPWR
- wire segments 134 -> 749
- no-connect marks 17 -> 15
Other:
- note added: "LED MATRIX"
- note added: "REF - Datasheet of IS31FL3731"
- moved on the sheet: C10, C11, C7, C8, C9, D145, FID1, FID2, FID3, H1, H2, H3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

Commit message: Gerbers for first prototype production
Parts:
- added H5, H6: Mouse Bites, Joels KiCad Footprint Library:Mouse_Bite_5mm_Wide, symbol Mechanical:MountingHole
- added H7, H8, H9: JLCPCB Mounting Hole, Joels KiCad Footprint Library:JCLPCB_Tooling_Hole, symbol Mechanical:MountingHole
Changed lines of the file:
@@
 Wire Wire Line
 	9950 2650 10300 2650
+$Comp
+L Mechanical:MountingHole H5
+U 1 1 62A5CDC2
+P 9850 6750
+F 0 "H5" H 9950 6796 50  0000 L CNN
+F 1 "Mouse Bites" H 9950 6705 50  0000 L CNN
+F 2 "Joels KiCad Footprint Library:Mouse_Bite_5mm_Wide" H 9850 6750 50  0001 C CNN
+F 3 "~" H 9850 6750 50  0001 C CNN
+	1    9850 6750
+	1    0    0    -1
+$EndComp
+$Comp
+L Mechanical:MountingHole H6
+U 1 1 62A5D9CF
+P 9850 7000
+F 0 "H6" H 9950 7046 50  0000 L CNN
+F 1 "Mouse Bites" H 9950 6955 50  0000 L CNN
+F 2 "Joels KiCad Footprint Library:Mouse_Bite_5mm_Wide" H 9850 7000 50  0001 C CNN
+F 3 "~" H 9850 7000 50  0001 C CNN
+	1    9850 7000
+	1    0    0    -1
+$EndComp
+$Comp
+L Mechanical:MountingHole H7
+U 1 1 61B38826
+P 9850 7550
+F 0 "H7" H 9950 7596 50  0000 L CNN
+F 1 "JLCPCB Mounting Hole" H 9950 7505 50  0000 L CNN
+F 2 "Joels KiCad Footprint Library:JCLPCB_Tooling_Hole" H 9850 7550 50  0001 C CNN
+F 3 "~" H 9850 7550 50  0001 C CNN
+	1    9850 7550
+	1    0    0    -1
+$EndComp
+$Comp
+L Mechanical:MountingHole H8
+U 1 1 61D1A081
+P 9850 7850
+F 0 "H8" H 9950 7896 50  0000 L CNN
+F 1 "JLCPCB Mounting Hole" H 9950 7805 50  0000 L CNN
+F 2 "Joels KiCad Footprint Library:JCLPCB_Tooling_Hole" H 9850 7850 50  0001 C CNN
+F 3 "~" H 9850 7850 50  0001 C CNN
+	1    9850 7850
+	1    0    0    -1
+$EndComp
+$Comp
+L Mechanical:MountingHole H9
+U 1 1 61DBC4A5
+P 9850 8150
+F 0 "H9" H 9950 8196 50  0000 L CNN
+F 1 "JLCPCB Mounting Hole" H 9950 8105 50  0000 L CNN
+F 2 "Joels KiCad Footprint Library:JCLPCB_Tooling_Hole" H 9850 8150 50  0001 C CNN
+F 3 "~" H 9850 8150 50  0001 C CNN
+	1    9850 8150
+	1    0    0    -1
+$EndComp
 $EndSCHEMATC

Commit message: Updated blinky schematic (ARM) for latest technology
Parts:
- removed D1.1, D1.10, D1.11, D1.12, D1.13, D1.14, D1.15, D1.16, D1.2, D1.3, D1.4, D1.5, D1.6, D1.7, D1.8, D1.9, D2.1, D2.10, D2.11, D2.12, D2.13, D2.14, D2.15, D2.16, D2.2, D2.3, D2.4, D2.5, D2.6, D2.7, D2.8, D2.9, D3.1, D3.10, D3.11, D3.12, D3.13, D3.14, D3.15, D3.16, D3.2, D3.3, D3.4, D3.5, D3.6, D3.7, D3.8, D3.9, D4.1, D4.10, D4.11, D4.12, D4.13, D4.14, D4.15, D4.16, D4.2, D4.3, D4.4, D4.5, D4.6, D4.7, D4.8, D4.9, D5.1, D5.10, D5.11, D5.12, D5.13, D5.14, D5.15, D5.16, D5.2, D5.3, D5.4, D5.5, D5.6, D5.7, D5.8, D5.9, D6.1, D6.10, D6.11, D6.12, D6.13, D6.14, D6.15, D6.16, D6.2, D6.3, D6.4, D6.5, D6.6, D6.7, D6.8, D6.9, D7.1, D7.10, D7.11, D7.12, D7.13, D7.14, D7.15, D7.16, D7.2, D7.3, D7.4, D7.5, D7.6, D7.7, D7.8, D7.9, D8.1, D8.10, D8.11, D8.12, D8.13, D8.14, D8.15, D8.16, D8.2, D8.3, D8.4, D8.5, D8.6, D8.7, D8.8, D8.9, D9.1, D9.10, D9.11, D9.12, D9.13, D9.14, D9.15, D9.16, D9.2, D9.3, D9.4, D9.5, D9.6, D9.7, D9.8, D9.9: LED, Joels KiCad Footprint Library:LED_0603_For_Blinky, symbol Device:LED
- removed FID1, FID2, FID3: Fiducial, Fiducial:Fiducial_1mm_Mask2mm, symbol Mechanical:Fiducial
- removed H1, H2, H3, H4: MountingHole, MountingHole:MountingHole_2mm, symbol Mechanical:MountingHole
- removed H5, H6: Mouse Bites, Joels KiCad Footprint Library:Mouse_Bite_5mm_Wide, symbol Mechanical:MountingHole
- removed H7, H8, H9: JLCPCB Mounting Hole, Joels KiCad Footprint Library:JCLPCB_Tooling_Hole, symbol Mechanical:MountingHole
- removed J2: NEOPIXEL, Joels KiCad Footprint Library:Debug_Pad_01x03, symbol Connector_Generic:Conn_01x03
- removed SW2: POWER, Joels KiCad Footprint Library:CK-JS102011JAQN-0-0-MFG, symbol Switch:SW_SPDT
- removed U3: TSOP75438WTT, Joels KiCad Footprint Library:TSOP75438WTT, symbol Joels_KiCad_Symbol_Library:TSOP754xxW
- added IC1: TSOP36438TT, Joels KiCad Footprint Library:TSOP36438TT, symbol Joels_KiCad_Symbol_Library:TSOP36438TT
- added J3: CA1-9, Connector_PinHeader_2.54mm:PinHeader_1x09_P2.54mm_Vertical, symbol Connector:Conn_01x09_Female
- added J4: CB1-9, Connector_PinHeader_2.54mm:PinHeader_1x09_P2.54mm_Vertical, symbol Connector:Conn_01x09_Female
- added S1: JS202011JCQN, Joels KiCad Footprint Library:CK-JS202011JCQN, symbol Joels_KiCad_Symbol_Library:JS202011JCQN
- J1: footprint Joels KiCad Footprint Library:Debug_Pad_02x05 -> Joels KiCad Footprint Library:SOIC_clipProgSmall; symbol Connector_Generic:Conn_02x05_Counter_Clockwise -> Connector_Generic:Conn_02x04_Counter_Clockwise
Connections:
- net labels added: A7, VBUS
- net labels removed: D+, D-, NEOPIX, NEOPWR, USB5V
- wire segments 749 -> 156
- no-connect marks 15 -> 22
Other:
- note added: "SOIC-8 CLIP FLASH AND TEST"
- note removed: "DEBUG, SETUP, TEST PADS"
- note removed: "REF - Datasheet of IS31FL3731"
- moved on the sheet: C7, D145, Q1, R3, R4, SW1

Commit message: routing this board here
Parts:
- added D1.1, D1.10, D1.11, D1.12, D1.13, D1.14, D1.15, D1.16, D1.2, D1.3, D1.4, D1.5, D1.6, D1.7, D1.8, D1.9, D2.1, D2.10, D2.11, D2.12, D2.13, D2.14, D2.15, D2.16, D2.2, D2.3, D2.4, D2.5, D2.6, D2.7, D2.8, D2.9, D3.1, D3.10, D3.11, D3.12, D3.13, D3.14, D3.15, D3.16, D3.2, D3.3, D3.4, D3.5, D3.6, D3.7, D3.8, D3.9, D4.1, D4.10, D4.11, D4.12, D4.13, D4.14, D4.15, D4.16, D4.2, D4.3, D4.4, D4.5, D4.6, D4.7, D4.8, D4.9, D5.1, D5.10, D5.11, D5.12, D5.13, D5.14, D5.15, D5.16, D5.2, D5.3, D5.4, D5.5, D5.6, D5.7, D5.8, D5.9, D6.1, D6.10, D6.11, D6.12, D6.13, D6.14, D6.15, D6.16, D6.2, D6.3, D6.4, D6.5, D6.6, D6.7, D6.8, D6.9, D7.1, D7.10, D7.11, D7.12, D7.13, D7.14, D7.15, D7.16, D7.2, D7.3, D7.4, D7.5, D7.6, D7.7, D7.8, D7.9, D8.1, D8.10, D8.11, D8.12, D8.13, D8.14, D8.15, D8.16, D8.2, D8.3, D8.4, D8.5, D8.6, D8.7, D8.8, D8.9, D9.1, D9.10, D9.11, D9.12, D9.13, D9.14, D9.15, D9.16, D9.2, D9.3, D9.4, D9.5, D9.6, D9.7, D9.8, D9.9: LED, Joels KiCad Footprint Library:LED_0603_For_Blinky, symbol Device:LED
Connections:
- net CA1: now also D1.1.1 (K), D1.2.1 (K), D1.3.1 (K), D1.4.1 (K), D1.5.1 (K), D1.6.1 (K), D1.7.1 (K), D1.8.1 (K), D2.1.2 (A), D3.1.2 (A), D4.1.2 (A), D5.1.2 (A), D6.1.2 (A), D7.1.2 (A), D8.1.2 (A), D9.1.2 (A)
- net CA2: now also D1.1.2 (A), D2.1.1 (K), D2.2.1 (K), D2.3.1 (K), D2.4.1 (K), D2.5.1 (K), D2.6.1 (K), D2.7.1 (K), D2.8.1 (K), D3.2.2 (A), D4.2.2 (A), D5.2.2 (A), D6.2.2 (A), D7.2.2 (A), D8.2.2 (A), D9.2.2 (A)
- net CA3: now also D1.2.2 (A), D2.2.2 (A), D3.1.1 (K), D3.2.1 (K), D3.3.1 (K), D3.4.1 (K), D3.5.1 (K), D3.6.1 (K), D3.7.1 (K), D3.8.1 (K), D4.3.2 (A), D5.3.2 (A), D6.3.2 (A), D7.3.2 (A), D8.3.2 (A), D9.3.2 (A)
- net CA4: now also D1.3.2 (A), D2.3.2 (A), D3.3.2 (A), D4.1.1 (K), D4.2.1 (K), D4.3.1 (K), D4.4.1 (K), D4.5.1 (K), D4.6.1 (K), D4.7.1 (K), D4.8.1 (K), D5.4.2 (A), D6.4.2 (A), D7.4.2 (A), D8.4.2 (A), D9.4.2 (A)
- net CA5: now also D1.4.2 (A), D2.4.2 (A), D3.4.2 (A), D4.4.2 (A), D5.1.1 (K), D5.2.1 (K), D5.3.1 (K), D5.4.1 (K), D5.5.1 (K), D5.6.1 (K), D5.7.1 (K), D5.8.1 (K), D6.5.2 (A), D7.5.2 (A), D8.5.2 (A), D9.5.2 (A)
- net CA6: now also D1.5.2 (A), D2.5.2 (A), D3.5.2 (A), D4.5.2 (A), D5.5.2 (A), D6.1.1 (K), D6.2.1 (K), D6.3.1 (K), D6.4.1 (K), D6.5.1 (K), D6.6.1 (K), D6.7.1 (K), D6.8.1 (K), D7.6.2 (A), D8.6.2 (A), D9.6.2 (A)
- net CA7: now also D1.6.2 (A), D2.6.2 (A), D3.6.2 (A), D4.6.2 (A), D5.6.2 (A), D6.6.2 (A), D7.1.1 (K), D7.2.1 (K), D7.3.1 (K), D7.4.1 (K), D7.5.1 (K), D7.6.1 (K), D7.7.1 (K), D7.8.1 (K), D8.7.2 (A), D9.7.2 (A)
- net CA8: now also D1.7.2 (A), D2.7.2 (A), D3.7.2 (A), D4.7.2 (A), D5.7.2 (A), D6.7.2 (A), D7.7.2 (A), D8.1.1 (K), D8.2.1 (K), D8.3.1 (K), D8.4.1 (K), D8.5.1 (K), D8.6.1 (K), D8.7.1 (K), D8.8.1 (K), D9.8.2 (A)
- net CA9: now also D1.8.2 (A), D2.8.2 (A), D3.8.2 (A), D4.8.2 (A), D5.8.2 (A), D6.8.2 (A), D7.8.2 (A), D8.8.2 (A), D9.1.1 (K), D9.2.1 (K), D9.3.1 (K), D9.4.1 (K), D9.5.1 (K), D9.6.1 (K), D9.7.1 (K), D9.8.1 (K)
- net CB1: now also D1.10.1 (K), D1.11.1 (K), D1.12.1 (K), D1.13.1 (K), D1.14.1 (K), D1.15.1 (K), D1.16.1 (K), D1.9.1 (K), D2.9.2 (A), D3.9.2 (A), D4.9.2 (A), D5.9.2 (A), D6.9.2 (A), D7.9.2 (A), D8.9.2 (A), D9.9.2 (A)
- net CB2: now also D1.9.2 (A), D2.10.1 (K), D2.11.1 (K), D2.12.1 (K), D2.13.1 (K), D2.14.1 (K), D2.15.1 (K), D2.16.1 (K), D2.9.1 (K), D3.10.2 (A), D4.10.2 (A), D5.10.2 (A), D6.10.2 (A), D7.10.2 (A), D8.10.2 (A), D9.10.2 (A)
- net CB3: now also D1.10.2 (A), D2.10.2 (A), D3.10.1 (K), D3.11.1 (K), D3.12.1 (K), D3.13.1 (K), D3.14.1 (K), D3.15.1 (K), D3.16.1 (K), D3.9.1 (K), D4.11.2 (A), D5.11.2 (A), D6.11.2 (A), D7.11.2 (A), D8.11.2 (A), D9.11.2 (A)
- net CB4: now also D1.11.2 (A), D2.11.2 (A), D3.11.2 (A), D4.10.1 (K), D4.11.1 (K), D4.12.1 (K), D4.13.1 (K), D4.14.1 (K), D4.15.1 (K), D4.16.1 (K), D4.9.1 (K), D5.12.2 (A), D6.12.2 (A), D7.12.2 (A), D8.12.2 (A), D9.12.2 (A)
- net CB5: now also D1.12.2 (A), D2.12.2 (A), D3.12.2 (A), D4.12.2 (A), D5.10.1 (K), D5.11.1 (K), D5.12.1 (K), D5.13.1 (K), D5.14.1 (K), D5.15.1 (K), D5.16.1 (K), D5.9.1 (K), D6.13.2 (A), D7.13.2 (A), D8.13.2 (A), D9.13.2 (A)
- net CB6: now also D1.13.2 (A), D2.13.2 (A), D3.13.2 (A), D4.13.2 (A), D5.13.2 (A), D6.10.1 (K), D6.11.1 (K), D6.12.1 (K), D6.13.1 (K), D6.14.1 (K), D6.15.1 (K), D6.16.1 (K), D6.9.1 (K), D7.14.2 (A), D8.14.2 (A), D9.14.2 (A)
- net CB7: now also D1.14.2 (A), D2.14.2 (A), D3.14.2 (A), D4.14.2 (A), D5.14.2 (A), D6.14.2 (A), D7.10.1 (K), D7.11.1 (K), D7.12.1 (K), D7.13.1 (K), D7.14.1 (K), D7.15.1 (K), D7.16.1 (K), D7.9.1 (K), D8.15.2 (A), D9.15.2 (A)
- net CB8: now also D1.15.2 (A), D2.15.2 (A), D3.15.2 (A), D4.15.2 (A), D5.15.2 (A), D6.15.2 (A), D7.15.2 (A), D8.10.1 (K), D8.11.1 (K), D8.12.1 (K), D8.13.1 (K), D8.14.1 (K), D8.15.1 (K), D8.16.1 (K), D8.9.1 (K), D9.16.2 (A)
- net CB9: now also D1.16.2 (A), D2.16.2 (A), D3.16.2 (A), D4.16.2 (A), D5.16.2 (A), D6.16.2 (A), D7.16.2 (A), D8.16.2 (A), D9.10.1 (K), D9.11.1 (K), D9.12.1 (K), D9.13.1 (K), D9.14.1 (K), D9.15.1 (K), D9.16.1 (K), D9.9.1 (K)
- net CFILT: now reaches C8.1, U4.16 (C_FILT)
- net AD: now reaches R10.1, U4.18 (AD)
Other:
- note added: "REF - Datasheet of IS31FL3731"

Commit message: making good progress on the circuit board
Parts:
- renumbered S1 to SW2, IC1 to U3
Connections:
- net 2RST: now reaches C4.1, R1.2, R2.2, U1.26 (~RESET)
- net VDDCORE: now reaches C2.1, U1.29 (VDDCORE)
Changed lines of the file:
@@
 Wire Notes Line
 	850  7200 850  4850
-$Comp
-L Joels_KiCad_Symbol_Library:TSOP36438TT IC1
-U 1 1 629FCB03
-P 12450 5450
-F 0 "IC1" H 12842 4885 50  0000 C CNN
-F 1 "TSOP36438TT" H 12842 4976 50  0000 C CNN
-F 2 "Joels KiCad Footprint Library:TSOP36438TT" H 13300 5550 50  0001 L CNN
-F 3 "https://www.mouser.com/datasheet/2/427/tsop362-464348.pdf" H 13300 5450 50  0001 L CNN
-F 4 "Infrared Receivers" H 13300 5350 50  0001 L CNN "Description"
-F 5 "5.3" H 13300 5250 50  0001 L CNN "Height"
-F 6 "Vishay" H 13300 5150 50  0001 L CNN "Manufacturer_Name"
-F 7 "TSOP36438TT" H 13300 5050 50  0001 L CNN "Manufacturer_Part_Number"
-F 8 "78-TSOP36438TT" H 13300 4950 50  0001 L CNN "Mouser Part Number"
-F 9 "https://www.mouser.co.uk/ProductDetail/Vishay-Semiconductors/TSOP36438TT?qs=b85dNVE93B5nGTLDDhv1%252Bg%3D%3D" H 13300 4850 50  0001 L CNN "Mouser Price/Stock"
-F 10 "TSOP36438TT" H 13300 4750 50  0001 L CNN "Arrow Part Number"
-F 11 "https://www.arrow.com/en/products/tsop36438tt/vishay?region=nac" H 13300 4650 50  0001 L CNN "Arrow Price/Stock"
-	1    12450 5450
-	-1   0    0    1
-$EndComp
 NoConn ~ 12450 5350
 Wire Wire Line
@@
 NoConn ~ 4100 2750
 $Comp
-L Joels_KiCad_Symbol_Library:JS202011JCQN S1
+L Joels_KiCad_Symbol_Library:JS202011JCQN SW2
 U 1 1 62AD4B38
 P 7850 1450
-F 0 "S1" H 7850 1817 50  0000 C CNN
+F 0 "SW2" H 7850 1817 50  0000 C CNN
 F 1 "JS202011JCQN" H 7850 1726 50  0000 C CNN
 F 2 "Joels KiCad Footprint Library:CK-JS202011JCQN" H 7850 1450 50  0001 L BNN
@@
 Text Label 12750 2250 0    50   ~ 0
 AD
+Text Label 4150 2150 0    50   ~ 0
+VDDCORE
+Text Label 4150 2450 0    50   ~ 0
+2RST
+$Comp
+L Joels_KiCad_Symbol_Library:TSOP36438TT U3
+U 1 1 629FCB03
+P 12450 5450
+F 0 "U3" H 12842 4885 50  0000 C CNN
+F 1 "TSOP36438TT" H 12842 4976 50  0000 C CNN
+F 2 "Joels KiCad Footprint Library:TSOP36438TT" H 13300 5550 50  0001 L CNN
+F 3 "https://www.mouser.com/datasheet/2/427/tsop362-464348.pdf" H 13300 5450 50  0001 L CNN
+F 4 "Infrared Receivers" H 13300 5350 50  0001 L CNN "Description"
+F 5 "5.3" H 13300 5250 50  0001 L CNN "Height"
+F 6 "Vishay" H 13300 5150 50  0001 L CNN "Manufacturer_Name"
+F 7 "TSOP36438TT" H 13300 5050 50  0001 L CNN "Manufacturer_Part_Number"
+F 8 "78-TSOP36438TT" H 13300 4950 50  0001 L CNN "Mouser Part Number"
+F 9 "https://www.mouser.co.uk/ProductDetail/Vishay-Semiconductors/TSOP36438TT?qs=b85dNVE93B5nGTLDDhv1%252Bg%3D%3D" H 13300 4850 50  0001 L CNN "Mouser Price/Stock"
+F 10 "TSOP36438TT" H 13300 4750 50  0001 L CNN "Arrow Part Number"
+F 11 "https://www.arrow.com/en/products/tsop36438tt/vishay?region=nac" H 13300 4650 50  0001 L CNN "Arrow Price/Stock"
+	1    12450 5450
+	-1   0    0    1
+$EndComp
 $EndSCHEMATC

Commit message: mousebite improvements
Parts:
- added H1, H2, H3, H4: Mouse Bite, Joels KiCad Footprint Library:Mouse_Bite_For_Clipper, symbol Mechanical:MountingHole
Changed lines of the file:
@@
 	-1   0    0    1
 $EndComp
+$Comp
+L Mechanical:MountingHole H1
+U 1 1 61EFA092
+P 1650 8100
+F 0 "H1" H 1750 8146 50  0000 L CNN
+F 1 "Mouse Bite" H 1750 8055 50  0000 L CNN
+F 2 "Joels KiCad Footprint Library:Mouse_Bite_For_Clipper" H 1650 8100 50  0001 C CNN
+F 3 "~" H 1650 8100 50  0001 C CNN
+	1    1650 8100
+	1    0    0    -1
+$EndComp
+$Comp
+L Mechanical:MountingHole H2
+U 1 1 61EFA5CA
+P 1650 8350
+F 0 "H2" H 1750 8396 50  0000 L CNN
+F 1 "Mouse Bite" H 1750 8305 50  0000 L CNN
+F 2 "Joels KiCad Footprint Library:Mouse_Bite_For_Clipper" H 1650 8350 50  0001 C CNN
+F 3 "~" H 1650 8350 50  0001 C CNN
+	1    1650 8350
+	1    0    0    -1
+$EndComp
+$Comp
+L Mechanical:MountingHole H3
+U 1 1 61F9A649
+P 1650 8600
+F 0 "H3" H 1750 8646 50  0000 L CNN
+F 1 "Mouse Bite" H 1750 8555 50  0000 L CNN
+F 2 "Joels KiCad Footprint Library:Mouse_Bite_For_Clipper" H 1650 8600 50  0001 C CNN
+F 3 "~" H 1650 8600 50  0001 C CNN
+	1    1650 8600
+	1    0    0    -1
+$EndComp
+$Comp
+L Mechanical:MountingHole H4
+U 1 1 6203A605
+P 1650 8850
+F 0 "H4" H 1750 8896 50  0000 L CNN
+F 1 "Mouse Bite" H 1750 8805 50  0000 L CNN
+F 2 "Joels KiCad Footprint Library:Mouse_Bite_For_Clipper" H 1650 8850 50  0001 C CNN
+F 3 "~" H 1650 8850 50  0001 C CNN
+	1    1650 8850
+	1    0    0    -1
+$EndComp
 $EndSCHEMATC

Commit message: lovely logo
Parts:
- added LOGO1: Future, Joels KiCad Footprint Library:logo-future, symbol Graphic:Logo_Open_Hardware_Small
- added LOGO2: Future, Joels KiCad Footprint Library:logo-turtles, symbol Graphic:Logo_Open_Hardware_Small
- C1: value 100uF 6.3V -> 100u
- C10, C11: value 10uF -> 10u
- C2, C7: value 1uF -> 1u
- C3, C4, C8, C9: value 0.1uF -> 0.1u
- C5: value 1.0uF -> 1.0u
- C6: value 2.2uF -> 2.2u
- R1: value 10kΩ -> 10K
- R2: value 330Ω -> 330
- R3: value 47Ω -> 47
- R4: value 470Ω -> 470
Changed lines of the file:
@@
 P 5050 3150
 F 0 "R1" H 5120 3196 50  0000 L CNN
-F 1 "10kΩ" H 5120 3105 50  0000 L CNN
+F 1 "10K" H 5120 3105 50  0000 L CNN
 F 2 "Resistor_SMD:R_0603_1608Metric" V 4980 3150 50  0001 C CNN
 F 3 "~" H 5050 3150 50  0001 C CNN
@@
 P 5400 3450
 F 0 "R2" V 5193 3450 50  0000 C CNN
-F 1 "330Ω" V 5284 3450 50  0000 C CNN
+F 1 "330" V 5284 3450 50  0000 C CNN
 F 2 "Resistor_SMD:R_0603_1608Metric" V 5330 3450 50  0001 C CNN
 F 3 "~" H 5400 3450 50  0001 C CNN
@@
 P 4950 3750
 F 0 "C4" H 5065 3796 50  0000 L CNN
-F 1 "0.1uF" H 5065 3705 50  0000 L CNN
+F 1 "0.1u" H 5065 3705 50  0000 L CNN
 F 2 "Capacitor_SMD:C_0603_1608Metric" H 4988 3600 50  0001 C CNN
 F 3 "~" H 4950 3750 50  0001 C CNN
@@
 P 5250 2300
 F 0 "C3" H 5365 2346 50  0000 L CNN
-F 1 "0.1uF" H 5365 2255 50  0000 L CNN
+F 1 "0.1u" H 5365 2255 50  0000 L CNN
 F 2 "Capacitor_SMD:C_0603_1608Metric" H 5288 2150 50  0001 C CNN
 F 3 "~" H 5250 2300 50  0001 C CNN
@@
 P 4900 2300
 F 0 "C2" H 5015 2346 50  0000 L CNN
-F 1 "1uF" H 5015 2255 50  0000 L CNN
+F 1 "1u" H 5015 2255 50  0000 L CNN
 F 2 "Capacitor_SMD:C_0603_1608Metric" H 4938 2150 50  0001 C CNN
 F 3 "~" H 4900 2300 50  0001 C CNN
@@
 P 6750 3850
 F 0 "C5" H 6865 3896 50  0000 L CNN
-F 1 "1.0uF" H 6865 3805 50  0000 L CNN
+F 1 "1.0u" H 6865 3805 50  0000 L CNN
 F 2 "Capacitor_SMD:C_0603_1608Metric" H 6788 3700 50  0001 C CNN
 F 3 "~" H 6750 3850 50  0001 C CNN
@@
 P 8500 3850
 F 0 "C6" H 8615 3896 50  0000 L CNN
-F 1 "2.2uF" H 8615 3805 50  0000 L CNN
+F 1 "2.2u" H 8615 3805 50  0000 L CNN
 F 2 "Capacitor_SMD:C_0603_1608Metric" H 8538 3700 50  0001 C CNN
 F 3 "~" H 8500 3850 50  0001 C CNN
@@
 P 7750 2150
 F 0 "C1" H 7865 2196 50  0000 L CNN
-F 1 "100uF 6.3V" H 7865 2105 50  0000 L CNN
+F 1 "100u" H 7865 2105 50  0000 L CNN
 F 2 "Capacitor_SMD:C_1206_3216Metric" H 7788 2000 50  0001 C CNN
 F 3 "~" H 7750 2150 50  0001 C CNN
@@
 P 14500 1600
 F 0 "C11" H 14592 1646 50  0000 L CNN
-F 1 "10uF" H 14592 1555 50  0000 L CNN
+F 1 "10u" H 14592 1555 50  0000 L CNN
 F 2 "Capacitor_SMD:C_0603_1608Metric" H 14500 1600 50  0001 C CNN
 F 3 "~" H 14500 1600 50  0001 C CNN
@@
 P 14100 1600
 F 0 "C10" H 14192 1646 50  0000 L CNN
-F 1 "10uF" H 14192 1555 50  0000 L CNN
+F 1 "10u" H 14192 1555 50  0000 L CNN
 F 2 "Capacitor_SMD:C_0603_1608Metric" H 14100 1600 50  0001 C CNN
 F 3 "~" H 14100 1600 50  0001 C CNN
@@
 P 13700 1600
 F 0 "C9" H 13792 1646 50  0000 L CNN
-F 1 "0.1uF" H 13792 1555 50  0000 L CNN
+F 1 "0.1u" H 13792 1555 50  0000 L CNN
 F 2 "Capacitor_SMD:C_0603_1608Metric" H 13700 1600 50  0001 C CNN
 F 3 "~" H 13700 1600 50  0001 C CNN
@@
 P 12400 3500
 F 0 "C8" H 12515 3546 50  0000 L CNN
-F 1 "0.1uF" H 12515 3455 50  0000 L CNN
+F 1 "0.1u" H 12515 3455 50  0000 L CNN
 F 2 "Capacitor_SMD:C_0603_1608Metric" H 12438 3350 50  0001 C CNN
 F 3 "~" H 12400 3500 50  0001 C CNN
@@
 P 12550 7500
 F 0 "R4" V 12343 7500 50  0000 C CNN
-F 1 "470Ω" V 12434 7500 50  0000 C CNN
+F 1 "470" V 12434 7500 50  0000 C CNN
 F 2 "Resistor_SMD:R_0603_1608Metric" V 12480 7500 50  0001 C CNN
 F 3 "~" H 12550 7500 50  0001 C CNN
@@
 P 13150 5400
 F 0 "C7" H 13265 5446 50  0000 L CNN
-F 1 "1uF" H 13265 5355 50  0000 L CNN
+F 1 "1u" H 13265 5355 50  0000 L CNN
 F 2 "Capacitor_SMD:C_0603_1608Metric" H 13188 5250 50  0001 C CNN
 F 3 "~" H 13150 5400 50  0001 C CNN
@@
 P 13500 5250
 F 0 "R3" V 13293 5250 50  0000 C CNN
-F 1 "47Ω" V 13384 5250 50  0000 C CNN
+F 1 "47" V 13384 5250 50  0000 C CNN
 F 2 "Resistor_SMD:R_0603_1608Metric" V 13430 5250 50  0001 C CNN
 F 3 "~" H 13500 5250 50  0001 C CNN
@@
 	1    0    0    -1
 $EndComp
+$Comp
+L Graphic:Logo_Open_Hardware_Small LOGO1
+U 1 1 61E27CB1
+P 3050 8100
+F 0 "LOGO1" H 3297 8171 50  0000 L CNN
+F 1 "Future" H 3297 8080 50  0000 L CNN
+F 2 "Joels KiCad Footprint Library:logo-future" H 3050 8100 50  0001 C CNN
+F 3 "~" H 3050 8100 50  0001 C CNN
+	1    3050 8100
+	1    0    0    -1
+$EndComp
+$Comp
+L Graphic:Logo_Open_Hardware_Small LOGO2
+U 1 1 61EC7BE6
+P 3050 8700
+F 0 "LOGO2" H 3297 8771 50  0000 L CNN
+F 1 "Future" H 3297 8680 50  0000 L CNN
+F 2 "Joels KiCad Footprint Library:logo-turtles" H 3050 8700 50  0001 C CNN
+F 3 "~" H 3050 8700 50  0001 C CNN
+	1    3050 8700
+	1    0    0    -1
+$EndComp

Commit message: more details
Parts:
- added FID1, FID2, FID3: Fiducial, Fiducial:Fiducial_1mm_Mask3mm, symbol Mechanical:Fiducial
- added H5, H6, H7, H8: MountingHole, Joels KiCad Footprint Library:JCLPCB_Tooling_Hole, symbol Mechanical:MountingHole
- added H9: Lanyard Hole, MountingHole:MountingHole_2.5mm_Pad_Via, symbol Mechanical:MountingHole
Changed lines of the file:
@@
+	1    0    0    -1
+$EndComp
+$Comp
+L Mechanical:Fiducial FID1
+U 1 1 620431A9
+P 1650 9500
+F 0 "FID1" H 1735 9546 50  0000 L CNN
+F 1 "Fiducial" H 1735 9455 50  0000 L CNN
+F 2 "Fiducial:Fiducial_1mm_Mask3mm" H 1650 9500 50  0001 C CNN
+F 3 "~" H 1650 9500 50  0001 C CNN
+	1    1650 9500
+	1    0    0    -1
+$EndComp
+$Comp
+L Mechanical:Fiducial FID2
+U 1 1 61D86C25
+P 1650 9700
+F 0 "FID2" H 1735 9746 50  0000 L CNN
+F 1 "Fiducial" H 1735 9655 50  0000 L CNN
+F 2 "Fiducial:Fiducial_1mm_Mask3mm" H 1650 9700 50  0001 C CNN
+F 3 "~" H 1650 9700 50  0001 C CNN
+	1    1650 9700
+	1    0    0    -1
+$EndComp
+$Comp
+L Mechanical:Fiducial FID3
+U 1 1 61E26B89
+P 1650 9900
+F 0 "FID3" H 1735 9946 50  0000 L CNN
+F 1 "Fiducial" H 1735 9855 50  0000 L CNN
+F 2 "Fiducial:Fiducial_1mm_Mask3mm" H 1650 9900 50  0001 C CNN
+F 3 "~" H 1650 9900 50  0001 C CNN
+	1    1650 9900
+	1    0    0    -1
+$EndComp
+$Comp
+L Mechanical:MountingHole H5
+U 1 1 61EE2AAC
+P 2900 9500
+F 0 "H5" H 3000 9546 50  0000 L CNN
+F 1 "MountingHole" H 3000 9455 50  0000 L CNN
+F 2 "Joels KiCad Footprint Library:JCLPCB_Tooling_Hole" H 2900 9500 50  0001 C CNN
+F 3 "~" H 2900 9500 50  0001 C CNN
+	1    2900 9500
+	1    0    0    -1
+$EndComp
+$Comp
+L Mechanical:MountingHole H6
+U 1 1 61EE30AB
+P 2900 9750
+F 0 "H6" H 3000 9796 50  0000 L CNN
+F 1 "MountingHole" H 3000 9705 50  0000 L CNN
+F 2 "Joels KiCad Footprint Library:JCLPCB_Tooling_Hole" H 2900 9750 50  0001 C CNN
+F 3 "~" H 2900 9750 50  0001 C CNN
+	1    2900 9750
+	1    0    0    -1
+$EndComp
+$Comp
+L Mechanical:MountingHole H7
+U 1 1 61F831CA
+P 2900 10000
+F 0 "H7" H 3000 10046 50  0000 L CNN
+F 1 "MountingHole" H 3000 9955 50  0000 L CNN
+F 2 "Joels KiCad Footprint Library:JCLPCB_Tooling_Hole" H 2900 10000 50  0001 C CNN
+F 3 "~" H 2900 10000 50  0001 C CNN
+	1    2900 10000
+	1    0    0    -1
+$EndComp
+$Comp
+L Mechanical:MountingHole H8
+U 1 1 620231D9
+P 2900 10250
+F 0 "H8" H 3000 10296 50  0000 L CNN
+F 1 "MountingHole" H 3000 10205 50  0000 L CNN
+F 2 "Joels KiCad Footprint Library:JCLPCB_Tooling_Hole" H 2900 10250 50  0001 C CNN
+F 3 "~" H 2900 10250 50  0001 C CNN
+	1    2900 10250
+	1    0    0    -1
+$EndComp
+$Comp
+L Mechanical:MountingHole H9
+U 1 1 620E81F6
+P 1650 10550
+F 0 "H9" H 1750 10596 50  0000 L CNN
+F 1 "Lanyard Hole" H 1750 10505 50  0000 L CNN
+F 2 "MountingHole:MountingHole_2.5mm_Pad_Via" H 1650 10550 50  0001 C CNN
+F 3 "~" H 1650 10550 50  0001 C CNN
+	1    1650 10550
 	1    0    0    -1
 $EndComp
